Commit message: Fix camera xyz & rpy

File: hands_on_ur5_description/urdf/hands_on_ur5.urdf.xacro (robot description, xacro)
@@ -43,5 +43,5 @@
     <xacro:property name = "camera_width" value ="0.04" />
     <joint name = "camera_joint" type = "fixed">
-        <origin xyz = "0.025 0.0 0.0" rpy="0 0 0" />
+        <origin xyz = "0.04 0.0 0.0" rpy="-1.57 -1.57 0" />
         <parent link = "ee_link" />
         <child link = "camera_link"/>

Commit message: Initial Commit

File: hands_on_ur5_description/urdf/hands_on_ur5.urdf.xacro (robot description, xacro)
@@ -43,5 +43,5 @@
     <xacro:property name = "camera_width" value ="0.04" />
     <joint name = "camera_joint" type = "fixed">
-        <origin xyz = "0.04 0.0 0.0" rpy="-1.57 -1.57 0" />
+        <origin xyz = "0.03 0.0 0.0" rpy="3.141 -1.5707 1.5707" />
         <parent link = "ee_link" />
         <child link = "camera_link"/>

Commit message: Fix distortion value miss

File: hands_on_ur5_description/urdf/hands_on_ur5.urdf.xacro (robot description, xacro)
@@ -43,5 +43,5 @@
     <xacro:property name = "camera_width" value ="0.04" />
     <joint name = "camera_joint" type = "fixed">
-        <origin xyz = "0.03 0.0 0.0" rpy="3.141 -1.5707 1.5707" />
+        <origin xyz = "0.03 0.0 0.0" rpy="3.141 0 1.5707" />
         <parent link = "ee_link" />
         <child link = "camera_link"/>
